Commit message: [airobo_description]URDFファイルをラズパイマウス参考に修正

File: 01_RaspberryPi/airobo_description/urdf/airobo_description.urdf (robot description, URDF)
Before this commit: robot airobo, 3 links, 2 joints
Links:
- removed link front_caster
- added link left_wheel; visual cylinder length=0.01 radius=0.045
- added link rear_caster; visual sphere radius=0.016
- added link right_wheel; visual cylinder length=0.01 radius=0.045
- link base_link: geometry visual box size=0.205 0.153 0.108
Joints:
- added joint left_wheel_joint: type continuous, parent base_link, child left_wheel, origin xyz=0.0175 0.057 -0.021 rpy=-1.57 0 0, axis 0 0 1
- added joint right_wheel_joint: type continuous, parent base_link, child right_wheel, origin xyz=0.0175 -0.057 -0.021 rpy=-1.57 0 0, axis 0 0 1
- joint base_joint: child base_footprint -> base_link; origin xyz=0.0 0.0 ${-(wheel_radius+wheel_zoff)} rpy=0 0 0 -> xyz=0 0 0.066; parent base_link -> base_footprint
- joint caster_joint: child front_caster -> rear_caster; origin xyz=${-caster_xoff} 0.0 ${-(base_height/2)} rpy=0 0 0 -> xyz=-0.0635 0.0 -0.058 rpy=0 0 0

Commit message: [airobo_description]URDFの修正

File: 01_RaspberryPi/airobo_description/urdf/airobo_description.urdf (robot description, URDF)
Before this commit: robot raspimouse, 5 links, 4 joints
Joints:
- joint left_wheel_joint: axis 0 0 1 -> 0 1 0; origin xyz=0.0175 0.057 -0.021 rpy=-1.57 0 0 -> xyz=0.0175 0.057 -0.021 rpy=0 0 0
- joint right_wheel_joint: axis 0 0 1 -> 0 1 0; origin xyz=0.0175 -0.057 -0.021 rpy=-1.57 0 0 -> xyz=0.0175 -0.057 -0.021 rpy=0 0 0

File: 01_RaspberryPi/airobo_description/urdf/airobo_description_bkup.urdf (robot description, URDF)
Before this commit: robot airobo, 3 links, 2 joints
Joints:
- joint base_joint: child base_footprint -> base_link; origin xyz=0.0 0.0 ${-(wheel_radius+wheel_zoff)} rpy=0 0 0 -> xyz=0 0 0.066; parent base_link -> base_footprint
